File: board/PCB/PCB.sch (KiCad schematic (older format))
At the start: 9 parts, among them K1 LolinD32pro_back, P1 PiezoBuzzerMH-FMD_back, P2 1.3\"OLED_Display, U1 SCD30_back

Commit message: PCB version 2
Parts:
- added J1: Conn_01x02_Female, symbol Connector:Conn_01x02_Female
Connections:
- net at K1.17 (GND), P1.3 (GND), P2.1 (GND)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: now also J1.1 (Pin_1), J1.2 (Pin_2)
Changed lines of the file:
@@
 	3100 3300 4300 3300
 Wire Wire Line
-	4300 2600 5150 2600
+	4300 2600 4800 2600
 Wire Wire Line
 	4300 3300 4300 2600
@@
 Wire Wire Line
 	6650 2050 4200 2050
+$Comp
+L Connector:Conn_01x02_Female J1
+U 1 1 60A2DD2C
+P 4800 2150
+F 0 "J1" V 4738 1962 50  0000 R CNN
+F 1 "Conn_01x02_Female" V 4647 1962 50  0000 R CNN
+F 2 "" H 4800 2150 50  0001 C CNN
+F 3 "~" H 4800 2150 50  0001 C CNN
+	1    4800 2150
+	0    -1   -1   0
+$EndComp
+Wire Wire Line
+	4900 2350 4900 2600
+Connection ~ 4900 2600
+Wire Wire Line
+	4900 2600 5150 2600
+Wire Wire Line
+	4800 2350 4800 2600
+Connection ~ 4800 2600
+Wire Wire Line
+	4800 2600 4900 2600
 $EndSCHEMATC

Commit message: PCB version 3.
Parts:
- J1: footprint (none) -> Connector_PinSocket_2.54mm:PinSocket_1x02_P2.54mm_Vertical
Changed lines of the file:
@@
 F 0 "J1" V 4738 1962 50  0000 R CNN
 F 1 "Conn_01x02_Female" V 4647 1962 50  0000 R CNN
-F 2 "" H 4800 2150 50  0001 C CNN
+F 2 "Connector_PinSocket_2.54mm:PinSocket_1x02_P2.54mm_Vertical" H 4800 2150 50  0001 C CNN
 F 3 "~" H 4800 2150 50  0001 C CNN
 	1    4800 2150

Commit message: board - PCB version 4
Parts:
- removed J1: Conn_01x02_Female, Connector_PinSocket_2.54mm:PinSocket_1x02_P2.54mm_Vertical, symbol Connector:Conn_01x02_Female
- added C1, C2: 0.1uF_Capacitor, Capacitor_THT:C_Axial_L3.8mm_D2.6mm_P10.00mm_Horizontal, symbol Device:C_Small
- added J1: GND_Out_1, Connector_PinHeader_2.54mm:PinHeader_1x01_P2.54mm_Vertical, symbol Connector:Conn_01x01_Male
- added J2: GND-Out_2, Connector_PinHeader_2.54mm:PinHeader_1x01_P2.54mm_Vertical, symbol Connector:Conn_01x01_Male
- renumbered U1 to IC1
Connections:
- net at IC1.2 (GND), K1.17 (GND), P1.3 (GND)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: now also C1.1, C2.2, J1.1 (Pin_1), J2.1 (Pin_1)
- net at IC1.1 (VDD), K1.1 (3V3), P1.1 (VCC)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: now also C1.2, C2.1
Other:
- note removed: "Achtung: Lolin und die andern Komponenten,\ndie auf die Rückseite sollen sind nicht spiegelverkehrt!\n->> Gelöst"
Changed lines of the file:
@@
 	0    1    1    0
 $EndComp
-Text Notes 7050 6850 0    50   ~ 10
-Achtung: Lolin und die andern Komponenten,\ndie auf die Rückseite sollen sind nicht spiegelverkehrt!\n->> Gelöst
 $Comp
 L 1.3_OLED_v.1.0:1.3"OLED_Display P2
@@
 $EndComp
 $Comp
-L SCD30:SCD30_back U1
+L SCD30:SCD30_back IC1
 U 1 1 6099312B
 P 8250 5400
-F 0 "U1" H 8022 5354 50  0000 R CNN
+F 0 "IC1" H 8022 5354 50  0000 R CNN
 F 1 "SCD30_back" H 8022 5445 50  0000 R CNN
 F 2 "MODULE_SCD30:MODULE_SCD30_back" H 8050 5450 50  0001 L BNN
@@
 	3200 2000 3200 1700
 Wire Wire Line
-	3200 1700 2250 1700
+	3200 1700 2400 1700
 Wire Wire Line
 	2250 1700 2250 3300
@@
 	3700 2950 3700 2600
 Wire Wire Line
-	3700 2600 3200 2600
+	3700 2600 3300 2600
 Wire Wire Line
 	3000 4650 3100 4650
@@
 Connection ~ 2250 3300
 Wire Wire Line
-	7950 4600 7300 4600
+	7950 4600 7850 4600
 Wire Wire Line
 	7300 4600 7300 5100
@@
 Wire Wire Line
 	3100 3300 4300 3300
-Wire Wire Line
-	4300 2600 4800 2600
 Wire Wire Line
 	4300 3300 4300 2600
@@
 Wire Wire Line
 	6650 2050 4200 2050
-$Comp
-L Connector:Conn_01x02_Female J1
-U 1 1 60A2DD2C
-P 4800 2150
-F 0 "J1" V 4738 1962 50  0000 R CNN
-F 1 "Conn_01x02_Female" V 4647 1962 50  0000 R CNN
-F 2 "Connector_PinSocket_2.54mm:PinSocket_1x02_P2.54mm_Vertical" H 4800 2150 50  0001 C CNN
-F 3 "~" H 4800 2150 50  0001 C CNN
-	1    4800 2150
-	0    -1   -1   0
-$EndComp
-Wire Wire Line
-	4900 2350 4900 2600
-Connection ~ 4900 2600
-Wire Wire Line
-	4900 2600 5150 2600
-Wire Wire Line
-	4800 2350 4800 2600
-Connection ~ 4800 2600
-Wire Wire Line
-	4800 2600 4900 2600
+Wire Wire Line
+	5150 2600 4750 2600
+$Comp
+L Connector:Conn_01x01_Male J1
+U 1 1 60A95CB2
+P 4500 2400
+F 0 "J1" V 4562 2444 50  0000 L CNN
+F 1 "GND_Out_1" V 4650 2000 50  0000 L CNN
+F 2 "Connector_PinHeader_2.54mm:PinHeader_1x01_P2.54mm_Vertical" H 4500 2400 50  0001 C CNN
+F 3 "~" H 4500 2400 50  0001 C CNN
+	1    4500 2400
+	0    1    1    0
+$EndComp
+Connection ~ 4500 2600
+Wire Wire Line
+	4500 2600 4300 2600
+$Comp
+L Connector:Conn_01x01_Male J2
+U 1 1 60A97242
+P 4750 2400
+F 0 "J2" V 4812 2444 50  0000 L CNN
+F 1 "GND-Out_2" V 4900 2400 50  0000 L CNN
+F 2 "Connector_PinHeader_2.54mm:PinHeader_1x01_P2.54mm_Vertical" H 4750 2400 50  0001 C CNN
+F 3 "~" H 4750 2400 50  0001 C CNN
+	1    4750 2400
+	0    1    1    0
+$EndComp
+Connection ~ 4750 2600
+Wire Wire Line
+	4750 2600 4500 2600
+$Comp
+L Device:C_Small C1
+U 1 1 60A9D12C
+P 2400 2300
+F 0 "C1" H 2492 2346 50  0000 L CNN
+F 1 "0.1uF_Capacitor" H 2492 2255 50  0000 L CNN
+F 2 "Capacitor_THT:C_Axial_L3.8mm_D2.6mm_P10.00mm_Horizontal" H 2400 2300 50  0001 C CNN
+F 3 "~" H 2400 2300 50  0001 C CNN
+	1    2400 2300
+	1    0    0    -1
+$EndComp
+$Comp
+L Device:C_Small C2
+U 1 1 60A9E4CE
+P 7950 4800
+F 0 "C2" H 7858 4754 50  0000 R CNN
+F 1 "0.1uF_Capacitor" H 7858 4845 50  0000 R CNN
+F 2 "Capacitor_THT:C_Axial_L3.8mm_D2.6mm_P10.00mm_Horizontal" H 7950 4800 50  0001 C CNN
+F 3 "~" H 7950 4800 50  0001 C CNN
+	1    7950 4800
+	-1   0    0    1
+$EndComp
+Wire Wire Line
+	7850 4900 7950 4900
+Connection ~ 7850 4600
+Wire Wire Line
+	7850 4600 7300 4600
+Wire Wire Line
+	2400 1700 2400 2200
+Connection ~ 2400 1700
+Wire Wire Line
+	2400 1700 2250 1700
+Wire Wire Line
+	3300 2600 3300 2700
+Wire Wire Line
+	3300 2700 2400 2700
+Wire Wire Line
+	2400 2700 2400 2400
+Connection ~ 3300 2600
+Wire Wire Line
+	3300 2600 3200 2600
+Connection ~ 7950 4700
+Wire Wire Line
+	7850 4600 7850 4900
 $EndSCHEMATC
